Commit message: Added simplified collision meshes.

File: robots/reactor_description.URDF (robot description, URDF)
Before this commit: robot reactor_description, 7 links, 6 joints
Links:
- link base_link: geometry collision mesh filename=package://reactor_description/meshes/base_link_hull.STL; visual mesh filename=package://reactor_description/meshes/base_link.STL
- link bicep_link: geometry collision mesh filename=package://reactor_description/meshes/bicep_link_hull.STL; visual mesh filename=package://reactor_description/meshes/bicep_link.STL
- link forearm_link: geometry collision mesh filename=package://reactor_description/meshes/forearm_link_hull.STL; visual mesh filename=package://reactor_description/meshes/forearm_link.STL
- link gripper_link: geometry collision mesh filename=package://reactor_description/meshes/gripper_link_hull.STL; visual mesh filename=package://reactor_description/meshes/gripper_link.STL
- link shoulder_link: geometry collision mesh filename=package://reactor_description/meshes/shoulder_link_hull.STL; visual mesh filename=package://reactor_description/meshes/shoulder_link.STL
- link wrist_1: geometry collision mesh filename=package://reactor_description/meshes/wrist_1_hull.STL; visual mesh filename=package://reactor_description/meshes/wrist_1.STL
- link wrist_2: geometry collision mesh filename=package://reactor_description/meshes/wrist_2_hull.STL; visual mesh filename=package://reactor_description/meshes/wrist_2.STL

Commit message: Added finger joint and finger links.

File: robots/reactor_description.URDF (robot description, URDF)
Before this commit: robot reactor_description, 7 links, 6 joints
Links:
- removed link gripper_link
- added link finger_link_1, mass 0.0078621; collision mesh filename=package://reactor_description/meshes/finger_link_hull.STL; visual mesh filename=package://reactor_description/meshes/finger_link.STL
- added link finger_link_2, mass 0.0078621; collision mesh filename=package://reactor_description/meshes/finger_link_hull.STL; visual mesh filename=package://reactor_description/meshes/finger_link.STL
- link wrist_2: mass 0.055706 -> 0.0648521292346638
Joints:
- removed joint gripper_joint
- added joint finger_joint: type prismatic, parent wrist_2, child finger_link_1, origin xyz=0.088882 -0.0187500 0.0012072 rpy=1.5708 -1.5572 -3.1416, axis 0 0 1, limit lower=0 upper=0.014 effort=1.5 velocity=0.01
- added joint finger_joint_2: type prismatic, parent wrist_2, child finger_link_2, origin xyz=0.088882 0.0187500 0.0012072 rpy=1.5708 1.5572 -1.4508E-15, axis 0 0 1, limit lower=0 upper=0.014 effort=1.5 velocity=0.01, mimic joint=finger_joint

Commit message: add in controllers for gazebo and update URDF to include tramissions

File: robots/reactor_description.URDF (robot description, URDF)
Before this commit: robot reactor_description, 8 links, 7 joints
Links:
- added link world
Joints:
- added joint grounding: type fixed, parent world, child base_link
